File: MiniSpec 2/Design Files/SensorStick-TSL2591/SensorStick-TSL2591.kicad_sch (KiCad schematic)
At the start: 6 parts, among them IC1 TSL25911FN, J1 TSM-104-02-S-DV-P-TR

Commit message: working on TSL2591 board
Parts:
- removed IC1: TSL25911FN, TSL25911FN, symbol SamacSys_Parts:TSL25911FN
- added IC1: TSL25913FN, TSL25913FN, symbol SamacSys_Parts:TSL25913FN
Connections:
- net +3V3: now also IC1.5 (VDD)
- net GND: now also IC1.3 (GND)
- net SCL: now also IC1.1 (SCL)
- net SDA: now also IC1.6 (SDA)
- net at R2.2: now also IC1.2 (INT)
Changed lines of the file:
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@@
   (junction (at 185.42 118.11) (diameter 0) (color 0 0 0 0)
   )
+  (junction (at 182.88 104.14) (diameter 0) (color 0 0 0 0)
+  )
   (junction (at 157.48 118.11) (diameter 0) (color 0 0 0 0)
   )
   (junction (at 95.25 96.52) (diameter 0) (color 0 0 0 0)
-  )
-  (junction (at 182.88 104.14) (diameter 0) (color 0 0 0 0)
   )
   (junction (at 157.48 104.14) (diameter 0) (color 0 0 0 0)
@@
     (pin "1")
   )
-  (symbol (lib_id "SamacSys_Parts:TSL25911FN") (at 157.48 104.14 0) (unit 1)
-    (in_bom yes) (on_board yes)
+  (symbol (lib_id "SamacSys_Parts:TSL25913FN") (at 157.48 104.14 0) (unit 1)
+    (in_bom yes) (on_board yes) (fields_autoplaced)
     (property "Reference" "IC1" (id 0) (at 170.18 96.52 0))
-    (property "Value" "TSL25911FN" (id 1) (at 170.18 99.06 0))
-    (property "Footprint" "TSL25911FN" (id 2) (at 165.1 93.98 0)
-      (effects (font (size 1.27 1.27)) (justify left))
-    )
-    (property "Datasheet" "http://ams.com/documents/20143/36005/TSL2591_DS000338_6-00.pdf" (id 3) (at 179.07 104.14 0)
-      (effects (font (size 1.27 1.27)) (justify left) hide)
-    )
-    (property "Description" "Sensitivity Ambient Light Sensor DFN6" (id 4) (at 179.07 106.68 0)
-      (effects (font (size 1.27 1.27)) (justify left) hide)
-    )
-    (property "Height" "0" (id 5) (at 179.07 109.22 0)
+    (property "Value" "TSL25913FN" (id 1) (at 170.18 99.06 0))
+    (property "Footprint" "TSL25913FN" (id 2) (at 179.07 101.6 0)
+      (effects (font (size 1.27 1.27)) (justify left) hide)
+    )
+    (property "Datasheet" "https://ams.com/documents/20143/36005/TSL2591_DS000338_6-00.pdf" (id 3) (at 179.07 104.14 0)
+      (effects (font (size 1.27 1.27)) (justify left) hide)
+    )
+    (property "Description" "Light to Digital Ambient Light Sensor Digital 3V 6-Pin DFN EP" (id 4) (at 179.07 106.68 0)
+      (effects (font (size 1.27 1.27)) (justify left) hide)
+    )
+    (property "Height" "1.15" (id 5) (at 179.07 109.22 0)
       (effects (font (size 1.27 1.27)) (justify left) hide)
     )
@@
       (effects (font (size 1.27 1.27)) (justify left) hide)
     )
-    (property "Manufacturer_Part_Number" "TSL25911FN" (id 7) (at 179.07 114.3 0)
-      (effects (font (size 1.27 1.27)) (justify left) hide)
-    )
-    (property "Mouser Part Number" "985-TSL25911FN" (id 8) (at 179.07 116.84 0)
-      (effects (font (size 1.27 1.27)) (justify left) hide)
-    )
-    (property "Mouser Price/Stock" "https://www.mouser.co.uk/ProductDetail/ams/TSL25911FN?qs=6irNfxKJ9AaiNMbaQmyIug%3D%3D" (id 9) (at 179.07 119.38 0)
-      (effects (font (size 1.27 1.27)) (justify left) hide)
-    )
-    (property "Arrow Part Number" "TSL25911FN" (id 10) (at 179.07 121.92 0)
-      (effects (font (size 1.27 1.27)) (justify left) hide)
-    )
-    (property "Arrow Price/Stock" "https://www.arrow.com/en/products/tsl25911fn/ams-ag?region=nac" (id 11) (at 179.07 124.46 0)
+    (property "Manufacturer_Part_Number" "TSL25913FN" (id 7) (at 179.07 114.3 0)
+      (effects (font (size 1.27 1.27)) (justify left) hide)
+    )
+    (property "Mouser Part Number" "985-TSL25913FN" (id 8) (at 179.07 116.84 0)
+      (effects (font (size 1.27 1.27)) (justify left) hide)
+    )
+    (property "Mouser Price/Stock" "https://www.mouser.co.uk/ProductDetail/ams/TSL25913FN?qs=abmNkq9no6CEMk6a7R%2FVTQ%3D%3D" (id 9) (at 179.07 119.38 0)
+      (effects (font (size 1.27 1.27)) (justify left) hide)
+    )
+    (property "Arrow Part Number" "TSL25913FN" (id 10) (at 179.07 121.92 0)
+      (effects (font (size 1.27 1.27)) (justify left) hide)
+    )
+    (property "Arrow Price/Stock" "https://www.arrow.com/en/products/tsl25913fn/ams-ag" (id 11) (at 179.07 124.46 0)
       (effects (font (size 1.27 1.27)) (justify left) hide)
     )
@@
       (reference "C1") (unit 1) (value "100nF") (footprint "Capacitor_SMD:C_1206_3216Metric_Pad1.42x1.75mm_HandSolder")
     )
-    (path "/1d736909-22b7-4469-8313-f42f4b653896"
-      (reference "IC1") (unit 1) (value "TSL25911FN") (footprint "TSL25911FN")
+    (path "/abd5b1f8-417b-4e4b-bb91-50def48c6e7b"
+      (reference "IC1") (unit 1) (value "TSL25913FN") (footprint "TSL25913FN")
     )
     (path "/00000000-0000-0000-0000-00005f3f1e47"

Commit message: added phone jack port for 25mm tube base
Parts:
- IC1: footprint TSL25913FN -> BinomicaLabs:TSL25911FN
- J1: footprint TSM-104-YY-ZZZ-DV-P-TR -> BinomicaLabs:TSM-104-YY-ZZZ-DV-P-TR
Changed lines of the file:
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@@
       (effects (font (size 1.27 1.27)) hide)
     )
-    (property "Footprint" "TSM-104-YY-ZZZ-DV-P-TR" (id 2) (at 111.76 88.9 0)
+    (property "Footprint" "BinomicaLabs:TSM-104-YY-ZZZ-DV-P-TR" (id 2) (at 111.76 88.9 0)
       (effects (font (size 1.27 1.27)) (justify left) hide)
     )
@@
     (property "Reference" "IC1" (id 0) (at 170.18 96.52 0))
     (property "Value" "TSL25913FN" (id 1) (at 170.18 99.06 0))
-    (property "Footprint" "TSL25913FN" (id 2) (at 179.07 101.6 0)
+    (property "Footprint" "BinomicaLabs:TSL25911FN" (id 2) (at 179.07 101.6 0)
       (effects (font (size 1.27 1.27)) (justify left) hide)
     )
@@
     )
     (path "/abd5b1f8-417b-4e4b-bb91-50def48c6e7b"
-      (reference "IC1") (unit 1) (value "TSL25913FN") (footprint "TSL25913FN")
+      (reference "IC1") (unit 1) (value "TSL25913FN") (footprint "BinomicaLabs:TSL25911FN")
     )
     (path "/00000000-0000-0000-0000-00005f3f1e47"
-      (reference "J1") (unit 1) (value "TSM-104-02-S-DV-P-TR") (footprint "TSM-104-YY-ZZZ-DV-P-TR")
+      (reference "J1") (unit 1) (value "TSM-104-02-S-DV-P-TR") (footprint "BinomicaLabs:TSM-104-YY-ZZZ-DV-P-TR")
     )
     (path "/00000000-0000-0000-0000-00005f4705d5"
