File: MiniSpec 2/Design Files/SpecPeripheral-I2C Bus Board/SpecPeripheral-I2C Bus Board v2.kicad_sch (KiCad schematic)
At the start: 14 parts, among them IC1 TCA9548APWR, J0 Conn_01x04_Female, J1 Conn_01x04_Female, J2 Conn_01x04_Female, J3 Conn_01x04_Female, J4 Conn_01x04_Female, J5 Conn_01x04_Female, J6 Conn_01x04_Female, J7 Conn_01x04_Female, J8 Conn_01x04_Female

Commit message: updated base board and made headway into I2C octopus board
Parts:
- added J?: SJ-43514-SMT-TR, SJ43514SMTTR, symbol SamacSys_Parts:SJ-43514-SMT-TR
- added R4, R5, R6: 10K, RESC3116X65N, symbol SamacSys_Parts:RC1206FR-0710KL
Connections:
- net GND: now also C1.1, IC1.12 (GND), R4.1, R5.1, R6.1; no longer C1.2, IC1.1 (A0), IC1.2 (A1), IC1.21 (A2), IC1.24 (VCC)
- net VCC: now also C1.2, IC1.24 (VCC); no longer C1.1, IC1.12 (GND)
- new net: IC1.1 (A0), R4.2
- new net: IC1.2 (A1), R5.2
- new net: IC1.21 (A2), R6.2
Other:
- moved on the sheet: R1
